File: mizet/mizet.kicad_sch (KiCad schematic)
At the start: 41 parts, among them J1 USB_C_Receptacle_USB2.0_16P, J2 Conn_01x04, J3 Conn_01x12, J4 Conn_01x12, SW1 RotaryEncoder_Switch_MP, SW2 SW_Push, SW3 SW_Push, SW4 SW_Push, SW5 SW_Push, U1 RP2040, U2 W25Q128JVS, U3 AMS1117-3.3, Y1 12MHz

Commit message: basic pcb
Parts:
- removed R5: 10k, Resistor_SMD:R_0402_1005Metric_Pad0.72x0.64mm_HandSolder, symbol Device:R
- removed U2: W25Q128JVS, Package_SO:SOIC-8_5.3x5.3mm_P1.27mm, symbol Memory_Flash:W25Q128JVS
- removed U3: AMS1117-3.3, Package_TO_SOT_SMD:SOT-223-3_TabPin2, symbol Regulator_Linear:AMS1117-3.3
- added D1: D_Schottky, Diode_SMD:D_SOD-123, symbol Device:D_Schottky
- added U1: XC6206PxxxMR, Package_TO_SOT_SMD:SOT-23-3, symbol Regulator_Linear:XC6206PxxxMR
- added U3: W25Q16JVSS, Package_SON:Winbond_USON-8-1EP_3x2mm_P0.5mm_EP0.2x1.6mm, symbol Memory_Flash:W25Q16JVSS
- J3, J4: footprint Connector_PinSocket_2.54mm:PinSocket_1x12_P2.54mm_Vertical -> Connector_PinHeader_2.54mm:PinHeader_1x12_P2.54mm_Vertical
- SW2, SW3, SW4, SW5: footprint Button_Switch_THT:SW_PUSH_1P1T_6x3.5mm_H4.3_APEM_MJTP1243 -> My_lib:tact_sw_smd
- U2: renamed from U1; footprint Package_DFN_QFN:QFN-56-1EP_7x7mm_P0.4mm_EP3.2x3.2mm -> My_lib:RP2040-QFN-56
- renumbered C7 to C10, C8 to C11, C9 to C12, C10 to C13, C11 to C14, C12 to C15, C13 to C16, C14 to C3, C15 to C4, C16 to C5, C3 to C6, C4 to C7, C5 to C8, C6 to C9, R3 to R1, R4 to R2, R1 to R3, R2 to R4, R6 to R5, R7 to R6, TP2 to TP1, TP1 to TP2
Connections:
- net +3V3: now also J4.3 (Pin_3), D1.2 (A), U1.2 (VO), U3.8 (VCC); no longer J3.3 (Pin_3)
- net GND: now also J4.2 (Pin_2), SW1.S1, SW2.1, SW3.1, SW4.1, SW5.1, U1.1 (GND), U3.4 (GND); no longer J3.2 (Pin_2), SW1.S2, SW2.2, SW3.2, SW4.2, SW5.2
- net GP0: now also J3.1 (Pin_1); no longer J4.1 (Pin_1)
- net GP1: now also J3.2 (Pin_2); no longer J4.2 (Pin_2)
- net GP10: now also J3.11 (Pin_11); no longer J4.11 (Pin_11)
- net GP11: now also J3.12 (Pin_12); no longer J4.12 (Pin_12)
- net GP2: now also J3.3 (Pin_3); no longer J4.3 (Pin_3)
- net GP25: now also J4.5 (Pin_5); no longer J3.8 (Pin_8)
- net GP26: now also J4.4 (Pin_4); no longer J3.7 (Pin_7)
- net GP3: now also J3.4 (Pin_4); no longer J4.4 (Pin_4)
- net GP4: now also J3.5 (Pin_5); no longer J4.5 (Pin_5)
- net GP5: now also J3.6 (Pin_6); no longer J4.6 (Pin_6)
- net GP6: now also J3.7 (Pin_7); no longer J4.7 (Pin_7)
- net GP7: now also J3.8 (Pin_8); no longer J4.8 (Pin_8)
- net GP8: now also J3.9 (Pin_9); no longer J4.9 (Pin_9)
- net GP9: now also J3.10 (Pin_10); no longer J4.10 (Pin_10)
- net QSPI_SCLK: now also U3.6 (CLK)
- net QSPI_SD0: now also U3.5 (DI/IO_{0})
- net QSPI_SD1: now also U3.2 (DO/IO_{1})
- net QSPI_SD2: now also U3.3 (~{WP}/IO_{2})
- net QSPI_SD3: now also U3.7 (~{HOLD}/~{RESET}/IO_{3})
- net QSPI_SS: now also U3.1 (~{CS})
- net RE_A: now also U2.18 (GPIO15); no longer U2.29 (GPIO18)
- net RE_B: now also U2.17 (GPIO14); no longer U2.30 (GPIO19)
- net RE_SW: now also SW1.S2, U2.27 (GPIO16); no longer SW1.S1, U2.31 (GPIO20)
- net SCL: now also U2.16 (GPIO13); no longer U2.28 (GPIO17)
- net SDA: now also U2.15 (GPIO12); no longer U2.27 (GPIO16)
- net SW_A: now also SW2.2, U2.41 (GPIO29_ADC3); no longer SW2.1, U2.32 (GPIO21)
- net SW_B: now also SW3.2, U2.40 (GPIO28_ADC2); no longer SW3.1, U2.34 (GPIO22)
- net SW_C: now also SW4.2, U2.39 (GPIO27_ADC1); no longer SW4.1, U2.35 (GPIO23)
- net SW_D: now also SW5.2, U2.28 (GPIO17); no longer SW5.1, U2.36 (GPIO24)
- net VBUS: now also J4.1 (Pin_1), D1.1 (K), U1.3 (VI); no longer J3.1 (Pin_1)
- removed net GP12: J3.12 (Pin_12), U2.15 (GPIO12)
- removed net GP13: J3.11 (Pin_11), U2.16 (GPIO13)
- removed net GP14: J3.10 (Pin_10), U2.17 (GPIO14)
- removed net GP15: J3.9 (Pin_9), U2.18 (GPIO15)
- removed net GP27: J3.6 (Pin_6), U2.39 (GPIO27_ADC1)
- removed net GP28: J3.5 (Pin_5), U2.40 (GPIO28_ADC2)
- removed net GP29: J3.4 (Pin_4), U2.41 (GPIO29_ADC3)
- new net GP18: J4.12 (Pin_12), U2.29 (GPIO18)
- new net GP19: J4.11 (Pin_11), U2.30 (GPIO19)
- new net GP20: J4.10 (Pin_10), U2.31 (GPIO20)
- new net GP21: J4.9 (Pin_9), U2.32 (GPIO21)
- new net GP22: J4.8 (Pin_8), U2.34 (GPIO22)
- new net GP23: J4.7 (Pin_7), U2.35 (GPIO23)
- new net GP24: J4.6 (Pin_6), U2.36 (GPIO24)
Other:
- moved on the sheet: C1, C10, C11, C12, C13, C14, C15, C16, C17, C2, C3, C4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

Commit message: update pcb
Parts:
- TP3, TP4: footprint TestPoint:TestPoint_Pad_D1.5mm -> Connector_PinHeader_2.54mm:PinHeader_1x01_P2.54mm_Horizontal
Connections:
- net GND: now also U3.9 (MP)
Changed lines of the file:
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@@
 	)
 	(junction
+		(at 104.14 105.41)
+		(diameter 0)
+		(color 0 0 0 0)
+	)
+	(junction
 		(at 93.98 85.09)
 		(diameter 0)
@@
 	(wire
 		(pts
+			(xy 104.14 105.41) (xy 106.68 105.41)
+		)
+		(stroke
+			(width 0)
+			(type default)
+		)
+	)
+	(wire
+		(pts
 			(xy 137.16 87.63) (xy 137.16 92.71)
 		)
@@
 			)
 		)
-		(property "Footprint" "TestPoint:TestPoint_Pad_D1.5mm"
+		(property "Footprint" "Connector_PinHeader_2.54mm:PinHeader_1x01_P2.54mm_Horizontal"
 			(at 166.37 105.41 0)
 			(effects
@@
 		(pin "4"
 		)
+		(pin "9"
+		)
 		(instances
 			(project ""
@@
 			)
 		)
-		(property "Footprint" "TestPoint:TestPoint_Pad_D1.5mm"
+		(property "Footprint" "Connector_PinHeader_2.54mm:PinHeader_1x01_P2.54mm_Horizontal"
 			(at 171.45 102.87 0)
 			(effects

Commit message: add mounting holes
Parts:
- removed TP2: ~{USB_BOOT}, TestPoint:TestPoint_Pad_D1.5mm, symbol Connector:TestPoint
- added H1, H2, H3: MountingHole, MountingHole:MountingHole_2.2mm_M2, symbol Mechanical:MountingHole
- added JP1: SolderJumper_2_Open, Jumper:SolderJumper-2_P1.3mm_Open_RoundedPad1.0x1.5mm, symbol Jumper:SolderJumper_2_Open
- renumbered TP3 to TP2, TP4 to TP3
Connections:
- net GND: now also JP1.1 (A)
- net at R5.2: now also JP1.2 (B)

Commit message: generate jlcpcb files
Parts:
- C1: value 10u -> 1u
- C2: value 22u -> 1u
- C4, C5: footprint Capacitor_SMD:C_0402_1005Metric_Pad0.74x0.62mm_HandSolder -> Capacitor_SMD:C_0603_1608Metric
Changed lines of the file:
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@@
 			)
 		)
-		(property "Footprint" "Capacitor_SMD:C_0402_1005Metric_Pad0.74x0.62mm_HandSolder"
+		(property "Footprint" "Capacitor_SMD:C_0603_1608Metric"
 			(at 147.32 86.6648 0)
 			(effects
@@
 			)
 		)
-		(property "Value" "22u"
+		(property "Value" "1u"
 			(at 130.81 43.1799 0)
 			(effects
@@
 			)
 		)
-		(property "Footprint" "Capacitor_SMD:C_0402_1005Metric_Pad0.74x0.62mm_HandSolder"
+		(property "Footprint" "Capacitor_SMD:C_0603_1608Metric"
 			(at 147.32 96.8248 0)
 			(effects
@@
 			)
 		)
-		(property "Value" "10u"
+		(property "Value" "1u"
 			(at 100.33 43.1799 0)
 			(effects
